File: TMC51604Axis/TMC51604Axis.sch (KiCad schematic (older format))
At the start: 44 parts, among them J1 +48Vin, J2 Stepper_conn, Q1 SUD08P06-155L, U1 AP2210-3.3V, U2 LM2937

Commit message: Bug fixes during first assembly
Parts:
- C1, C14, C2: symbol Device:C_Small -> TMC51604Axis-rescue:C_Small-Device
- C10, C11, C12, C13, C4, C6, C8, C9: symbol Device:C -> TMC51604Axis-rescue:C-Device
- C3, C7: symbol Device:CP -> TMC51604Axis-rescue:CP-Device
- C5: value 47nF -> 47nF/100V; symbol Device:C -> TMC51604Axis-rescue:C-Device
- D1: symbol Diode:1N4148W -> TMC51604Axis-rescue:1N4148W-Diode
- D2, D3: symbol Device:D_Zener -> TMC51604Axis-rescue:D_Zener-Device
- D4: symbol Device:LED -> TMC51604Axis-rescue:LED-Device
- D5: symbol Peters:LT1766 -> TMC51604Axis-rescue:LT1766-Peters
- D6: value D_Schottky -> SS34FA; symbol Device:D_Schottky -> TMC51604Axis-rescue:D_Schottky-Device
- F1: symbol Device:Fuse -> TMC51604Axis-rescue:Fuse-Device
- FB2: symbol Device:Ferrite_Bead -> TMC51604Axis-rescue:Ferrite_Bead-Device
- H1, H2, H3, H4: symbol Mechanical:MountingHole -> TMC51604Axis-rescue:MountingHole-Mechanical
- J1: symbol Connector:Conn_01x02_Female -> TMC51604Axis-rescue:Conn_01x02_Female-Connector
- J2: symbol Connector:Screw_Terminal_01x04 -> TMC51604Axis-rescue:Screw_Terminal_01x04-Connector
- L1: symbol Device:L -> TMC51604Axis-rescue:L-Device
- Q1: symbol Transistor_FET:SUD08P06-155L -> TMC51604Axis-rescue:SUD08P06-155L-Transistor_FET
- R1, R3, R4: symbol Device:R -> TMC51604Axis-rescue:R-Device
- R2, R5, R6: symbol Device:R_Small -> TMC51604Axis-rescue:R_Small-Device
- TP1, TP2, TP4, TP5, TP6, TP7: symbol Connector:TestPoint -> TMC51604Axis-rescue:TestPoint-Connector
- U1: symbol Peters:AP2210-3.3V -> TMC51604Axis-rescue:AP2210-3.3V-Peters
- U2: symbol Peters:LM2937 -> TMC51604Axis-rescue:LM2937-Peters
Changed lines of the file:
@@
 $EndSheet
 $Comp
-L Connector:Conn_01x02_Female J1
+L TMC51604Axis-rescue:Conn_01x02_Female-Connector J1
 U 1 1 5ECB9EB8
 P 900 1150
@@
 	5600 5200 5300 5200
 $Comp
-L Device:C C5
+L TMC51604Axis-rescue:C-Device C5
 U 1 1 5ED05A0D
 P 2550 1300
 F 0 "C5" H 2350 1300 50  0000 L CNN
-F 1 "47nF" H 2350 1150 50  0000 L CNN
+F 1 "47nF/100V" H 2350 1150 50  0000 L CNN
 F 2 "peters:C_0805_peter" H 2588 1150 50  0001 C CNN
 F 3 "~" H 2550 1300 50  0001 C CNN
@@
 $EndComp
 $Comp
-L Transistor_FET:SUD08P06-155L Q1
+L TMC51604Axis-rescue:SUD08P06-155L-Transistor_FET Q1
 U 1 1 5ED0C6B9
 P 1800 1150
@@
 $EndComp
 $Comp
-L Device:D_Zener D3
+L TMC51604Axis-rescue:D_Zener-Device D3
 U 1 1 5ED0DCA9
 P 2100 1300
@@
 $EndComp
 $Comp
-L Device:R R3
+L TMC51604Axis-rescue:R-Device R3
 U 1 1 5ED15B9A
 P 1800 1600
@@
 Connection ~ 1800 1750
 $Comp
-L Device:R R1
+L TMC51604Axis-rescue:R-Device R1
 U 1 1 5ED28378
 P 3050 1050
@@
 $EndComp
 $Comp
-L Connector:TestPoint TP1
+L TMC51604Axis-rescue:TestPoint-Connector TP1
 U 1 1 5ED2B264
 P 2550 950
@@
 $EndComp
 $Comp
-L Connector:TestPoint TP2
+L TMC51604Axis-rescue:TestPoint-Connector TP2
 U 1 1 5ED2BA57
 P 3350 950
@@
 Connection ~ 3350 1050
 $Comp
-L Device:LED D4
+L TMC51604Axis-rescue:LED-Device D4
 U 1 1 5EFA7135
 P 3550 1300
@@
 $EndComp
 $Comp
-L Device:R R4
+L TMC51604Axis-rescue:R-Device R4
 U 1 1 5EFA90DA
 P 3550 1600
@@
 Connection ~ 2550 1750
 $Comp
-L Device:Fuse F1
+L TMC51604Axis-rescue:Fuse-Device F1
 U 1 1 5EFACFB0
 P 1250 1050
@@
 	1400 1150 1100 1150
 $Comp
-L power:GND #PWR06
+L TMC51604Axis-rescue:GND-power #PWR06
 U 1 1 5EC840BA
 P 4000 1400
@@
 	4000 1400 4000 1350
 $Comp
-L Peters:LT1766 D5
+L TMC51604Axis-rescue:LT1766-Peters D5
 U 1 1 5EC24277
 P 5600 1300
@@
 $EndComp
 $Comp
-L power:GND #PWR09
+L TMC51604Axis-rescue:GND-power #PWR09
 U 1 1 5EC2FFA1
 P 5600 1950
@@
 $EndComp
 $Comp
-L Device:L L1
+L TMC51604Axis-rescue:L-Device L1
 U 1 1 5EC33164
 P 6800 1200
@@
 $EndComp
 $Comp
-L Device:C_Small C1
+L TMC51604Axis-rescue:C_Small-Device C1
 U 1 1 5EC34588
 P 6400 1100
@@
 $EndComp
 $Comp
-L Device:D_Schottky D6
+L TMC51604Axis-rescue:D_Schottky-Device D6
 U 1 1 5EC365E4
 P 6400 1550
 F 0 "D6" V 6354 1630 50  0000 L CNN
-F 1 "D_Schottky" V 6445 1630 50  0000 L CNN
+F 1 "SS34FA" V 6445 1630 50  0000 L CNN
 F 2 "Diode_SMD:D_SOD-123F" H 6400 1550 50  0001 C CNN
 F 3 "~" H 6400 1550 50  0001 C CNN
@@
 	7000 1200 6950 1200
 $Comp
-L Device:R_Small R2
+L TMC51604Axis-rescue:R_Small-Device R2
 U 1 1 5EC4223F
 P 6250 1450
@@
 	5100 1500 4950 1500
 $Comp
-L power:GND #PWR05
+L TMC51604Axis-rescue:GND-power #PWR05
 U 1 1 5EC591D4
 P 5050 1350
@@
 	5100 1350 5050 1350
 $Comp
-L Diode:1N4148W D1
+L TMC51604Axis-rescue:1N4148W-Diode D1
 U 1 1 5EC5B891
 P 6350 850
@@
 $EndComp
 $Comp
-L Device:D_Zener D2
+L TMC51604Axis-rescue:D_Zener-Device D2
 U 1 1 5EC5D08E
 P 6750 850
@@
 Connection ~ 7200 1200
 $Comp
-L Device:CP C7
+L TMC51604Axis-rescue:CP-Device C7
 U 1 1 5EC7675D
 P 7200 1500
@@
 	6250 1550 6250 1600
 $Comp
-L Device:R_Small R5
+L TMC51604Axis-rescue:R_Small-Device R5
 U 1 1 5EC42B52
 P 6250 1700
@@
 	6250 1850 5600 1850
 $Comp
-L Device:C C4
+L TMC51604Axis-rescue:C-Device C4
 U 1 1 5EC82DDD
 P 4450 1200
@@
 Connection ~ 4450 1050
 $Comp
-L power:GND #PWR07
+L TMC51604Axis-rescue:GND-power #PWR07
 U 1 1 5EC8447E
 P 4450 1400
@@
 	4450 1400 4450 1350
 $Comp
-L Device:CP C3
+L TMC51604Axis-rescue:CP-Device C3
 U 1 1 5EC8F720
 P 4000 1200
-F 0 "C3" H 4118 1246 50  0000 L CNN
+F 0 "C3" H 3950 1450 50  0000 L CNN
 F 1 "10uF/100v" V 4200 850 50  0000 L CNN
 F 2 "Capacitor_SMD:CP_Elec_8x6.2" H 4038 1050 50  0001 C CNN
@@
 	4000 1050 4450 1050
 $Comp
-L Device:C C13
+L TMC51604Axis-rescue:C-Device C13
 U 1 1 5ECA4151
 P 4950 1650
@@
 Connection ~ 4950 1500
 $Comp
-L Device:R_Small R6
+L TMC51604Axis-rescue:R_Small-Device R6
 U 1 1 5ECAD316
 P 4750 1900
@@
 $EndComp
 $Comp
-L Device:C_Small C14
+L TMC51604Axis-rescue:C_Small-Device C14
 U 1 1 5ECAE19E
 P 4750 2150
@@
 	4750 2050 4750 2000
 $Comp
-L power:GND #PWR010
+L TMC51604Axis-rescue:GND-power #PWR010
 U 1 1 5ECB0DED
 P 4750 2350
@@
 	4750 2300 4750 2350
 $Comp
-L power:+48V #PWR01
+L TMC51604Axis-rescue:+48V-power #PWR01
 U 1 1 5ECB6C55
 P 4450 900
@@
 	4450 900  4450 1050
 $Comp
-L power:+48V #PWR011
+L TMC51604Axis-rescue:+48V-power #PWR011
 U 1 1 5ECBA302
 P 5550 4000
@@
 $EndComp
 $Comp
-L power:+12V #PWR012
+L TMC51604Axis-rescue:+12V-power #PWR012
 U 1 1 5ECBB50A
 P 5800 4000
@@
 	5300 4350 6100 4350
 $Comp
-L Peters:+3.3V #PWR013
+L TMC51604Axis-rescue:+3.3V-Peters #PWR013
 U 1 1 5ECF24FB
 P 6100 4000
@@
 $EndComp
 $Comp
-L Device:C C12
+L TMC51604Axis-rescue:C-Device C12
 U 1 1 5ECFF908
 P 9750 3050
@@
 $EndComp
 $Comp
-L Device:C C6
+L TMC51604Axis-rescue:C-Device C6
 U 1 1 5ED00402
 P 10150 2900
@@
 $EndComp
 $Comp
-L Device:C C11
+L TMC51604Axis-rescue:C-Device C11
 U 1 1 5ED00A27
 P 8250 3050
@@
 	9750 3400 9150 3400
 $Comp
-L Peters:+3.3V #PWR04
+L TMC51604Axis-rescue:+3.3V-Peters #PWR04
 U 1 1 5ED30E59
 P 10150 2750
@@
 	6100 4350 6100 4000
 $Comp
-L Peters:LM2937 U2
+L TMC51604Axis-rescue:LM2937-Peters U2
 U 1 1 5ED7FF5A
 P 7600 2650
@@
 	7500 3400 7950 3400
 $Comp
-L Device:C C9
+L TMC51604Axis-rescue:C-Device C9
 U 1 1 5ED94130
 P 7100 3050
@@
 $EndComp
 $Comp
-L Device:C C10
+L TMC51604Axis-rescue:C-Device C10
 U 1 1 5ED94E73
 P 7950 3050
@@
 	7950 3400 8250 3400
 $Comp
-L power:+5V #PWR03
+L TMC51604Axis-rescue:+5V-power #PWR03
 U 1 1 5EDA6039
 P 8250 2700
@@
 	8250 2700 8250 2750
 $Comp
-L Connector:Screw_Terminal_01x04 J2
+L TMC51604Axis-rescue:Screw_Terminal_01x04-Connector J2
 U 1 1 5EE4D43F
 P 5800 5000
@@
 Connection ~ 2550 1050
 $Comp
-L Device:C_Small C2
+L TMC51604Axis-rescue:C_Small-Device C2
 U 1 1 5ECF6516
 P 3050 1200
@@
 	2800 1050 2900 1050
 $Comp
-L power:+12V #PWR02
+L TMC51604Axis-rescue:+12V-power #PWR02
 U 1 1 5EC65390
 P 7600 1050
@@
 $EndSheet
 $Comp
-L Mechanical:MountingHole H1
+L TMC51604Axis-rescue:MountingHole-Mechanical H1
 U 1 1 5EDCC0E6
 P 10400 5650
@@
 $EndComp
 $Comp
-L Mechanical:MountingHole H2
+L TMC51604Axis-rescue:MountingHole-Mechanical H2
 U 1 1 5EDCC0EC
 P 10400 5850
@@
 $EndComp
 $Comp
-L Mechanical:MountingHole H3
+L TMC51604Axis-rescue:MountingHole-Mechanical H3
 U 1 1 5EDCC0F2
 P 10400 6050
@@
 $EndComp
 $Comp
-L Mechanical:MountingHole H4
+L TMC51604Axis-rescue:MountingHole-Mechanical H4
 U 1 1 5EDCC0F8
 P 10400 6250
@@
 $EndComp
 $Comp
-L Device:Ferrite_Bead FB2
+L TMC51604Axis-rescue:Ferrite_Bead-Device FB2
 U 1 1 5ED11BFB
 P 6800 2750
@@
 	7600 1050 7600 1200
 $Comp
-L power:+12V #PWR044
+L TMC51604Axis-rescue:+12V-power #PWR044
 U 1 1 5F1ED2CA
 P 6250 2650
@@
 	6250 2750 6250 2650
 $Comp
-L power:GND #PWR048
+L TMC51604Axis-rescue:GND-power #PWR048
 U 1 1 5F1FA36F
 P 7500 3400
@@
 	2900 4000 3900 4000
 $Comp
-L Peters:AP2210-3.3V U1
+L TMC51604Axis-rescue:AP2210-3.3V-Peters U1
 U 1 1 5F245C78
 P 9150 2550
@@
 $EndComp
 $Comp
-L power:GND #PWR0101
+L TMC51604Axis-rescue:GND-power #PWR0101
 U 1 1 5ECAFA60
 P 2550 1750
@@
 	2100 1050 2550 1050
 $Comp
-L Connector:TestPoint TP4
+L TMC51604Axis-rescue:TestPoint-Connector TP4
 U 1 1 5F8846DE
 P 8900 1250
@@
 $EndComp
 $Comp
-L Connector:TestPoint TP5
+L TMC51604Axis-rescue:TestPoint-Connector TP5
 U 1 1 5F8851C5
 P 9500 1250
@@
 $EndComp
 $Comp
-L Connector:TestPoint TP6
+L TMC51604Axis-rescue:TestPoint-Connector TP6
 U 1 1 5F885A15
 P 10100 1250
@@
 $EndComp
 $Comp
-L Connector:TestPoint TP7
+L TMC51604Axis-rescue:TestPoint-Connector TP7
 U 1 1 5F8973EF
 P 8450 1250
@@
 $EndComp
 $Comp
-L power:GND #PWR0102
+L TMC51604Axis-rescue:GND-power #PWR0102
 U 1 1 5F897905
 P 8450 1250
@@
 	7200 1200 7600 1200
 $Comp
-L power:+12V #PWR0103
+L TMC51604Axis-rescue:+12V-power #PWR0103
 U 1 1 5F8D8D2B
 P 9250 1250
@@
 	9250 1250 8900 1250
 $Comp
-L power:+5V #PWR0104
+L TMC51604Axis-rescue:+5V-power #PWR0104
 U 1 1 5F8DDF9A
 P 9900 1250
@@
 	9650 2750 10150 2750
 $Comp
-L Peters:+3.3V #PWR0105
+L TMC51604Axis-rescue:+3.3V-Peters #PWR0105
 U 1 1 5F8E2D13
 P 10500 1250
@@
 	10500 1250 10100 1250
 $Comp
-L Device:C C8
+L TMC51604Axis-rescue:C-Device C8
 U 1 1 5F8FCFC8
 P 7600 1500
