File: TMC51604Axis/TMC51604Axis.sch (KiCad schematic (older format))
At the start: 44 parts, among them J1 +48Vin, J2 Stepper_conn, Q1 SUD08P06-155L, U1 AP2210-3.3V, U2 LM2937

Commit message: First layout V2
Parts:
- removed C2: 10p, peters:C_0805_peter, symbol TMC51604Axis-rescue:C_Small-Device
- removed C5: 47nF/100V, peters:C_0805_peter, symbol TMC51604Axis-rescue:C-Device
- removed F1: Fuse, Fuse:Fuse_2512_6332Metric, symbol TMC51604Axis-rescue:Fuse-Device
- removed Q1: SUD08P06-155L, Package_TO_SOT_SMD:TO-252-2, symbol TMC51604Axis-rescue:SUD08P06-155L-Transistor_FET
- removed R1: 0R01, Resistor_SMD:R_2512_6332Metric, symbol TMC51604Axis-rescue:R-Device
- removed TP1, TP2: TestPoint, TestPoint:TestPoint_Pad_D1.5mm, symbol TMC51604Axis-rescue:TestPoint-Connector
- added J7: Stepper_conn, Connector_Phoenix_MSTB:PhoenixContact_MSTBA_2,5_4-G-5,08_1x04_P5.08mm_Horizontal, symbol TMC51604Axis-rescue:Screw_Terminal_01x04-Connector
- added Q5: SQJ481EP, Libs:PowerPAK SO-8L SINGLE, symbol Peters:SQJ481EP
- C3, C4: footprint Capacitor_SMD:CP_Elec_8x6.2 -> Capacitor_SMD:CP_Elec_8x10
- C8: footprint Capacitor_SMD:C_2010_5025Metric_Pad1.52x2.65mm_HandSolder -> Capacitor_SMD:C_1210_3225Metric_Pad1.33x2.70mm_HandSolder
- FB2: footprint Resistor_SMD:R_0805_2012Metric_Pad1.15x1.40mm_HandSolder -> Resistor_SMD:R_0805_2012Metric_Pad1.20x1.40mm_HandSolder
- TP4, TP5, TP6: footprint TestPoint:TestPoint_Pad_1.5x1.5mm -> TestPoint:TestPoint_THTPad_D1.0mm_Drill0.5mm
Connections:
- net +48V: now also D3.1 (K), Q5.1 (S), Q5.2 (S), Q5.3 (S)
- net MotorDrv1/StepperA: now also J2.4 (Pin_4), J7.4 (Pin_4); no longer J2.1 (Pin_1)
- net MotorDrv1/StepperB: now also J2.3 (Pin_3), J7.3 (Pin_3); no longer J2.2 (Pin_2)
- net MotorDrv1/StepperC: now also J2.2 (Pin_2), J7.2 (Pin_2); no longer J2.3 (Pin_3)
- net MotorDrv1/StepperD: now also J2.1 (Pin_1), J7.1 (Pin_1); no longer J2.4 (Pin_4)
- net at J1.2 (Pin_2): now also Q5.5 (D)
- net at D3.2 (A), R3.1: now also Q5.4 (G)
Other:
- moved on the sheet: D3, J1, R3

Commit message: sync
Changed lines of the file:
@@
 U 1 1 5EC24277
 P 5600 1300
-F 0 "D5" H 5650 1750 50  0000 C CNN
-F 1 "LT1766" H 5700 1400 50  0000 C CNN
+F 0 "D5" H 5625 1775 50  0000 C CNN
+F 1 "LT1766" H 5625 1684 50  0000 C CNN
 F 2 "Package_SO:TSSOP-16-1EP_4.4x5mm_P0.65mm" H 5600 1900 50  0001 C CNN
 F 3 "http://192.168.10.161/api/part_attachments/2499/getFile" H 5600 1900 50  0001 C CNN
