File: TMC51604Axis/Inputs.sch (KiCad schematic (older format))
At the start: 51 parts, among them J3 RJ45_Shielded, J4 EncCon1, J5 RJ45_Shielded, J6 EncCon2, U5 74LVC125, U6 74LVC125, U7 74LVC125

Commit message: Redone input section
Parts:
- added C46, C47: 100n, peters:C_0805_peter, symbol Device:C
- added R50: 20R, peters:R_0805_peter, symbol Device:R
Connections:
- net labels added: Signal_VCC
- net labels removed: CLK_raw, DIR_REFR_raw, DRV_ENN_raw, STEP_REFL_raw
- wire segments 153 -> 117
Other:
- note added: "Encoder interface"
- note removed: "Status LED's W. buffers"
- moved on the sheet: R31, R32, R33, R34, R35, R36, R37, R38, R39, R40, R41, R42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

Commit message: Bug fixes during first assembly
Parts:
- C42, C43, C44, C45, C46, C47: symbol Device:C -> TMC51604Axis-rescue:C-Device
- D11, D12, D13, D14, D15, D16, D17, D18, D19: symbol Device:LED -> TMC51604Axis-rescue:LED-Device
- D20, D21, D22, D23, D24, D25, D26, D27, D28, D29: symbol Diode:BAT54S -> TMC51604Axis-rescue:BAT54S-Diode
- J3, J5: symbol Connector:RJ45_Shielded -> TMC51604Axis-rescue:RJ45_Shielded-Connector
- J4, J6: symbol Connector:Screw_Terminal_01x03 -> TMC51604Axis-rescue:Screw_Terminal_01x03-Connector
- JP3: symbol Jumper:Jumper_3_Bridged12 -> TMC51604Axis-rescue:Jumper_3_Bridged12-Jumper
- R31, R32, R33, R34, R35, R36, R37, R38, R39, R40, R41, R42, R43, R44, R45, R46, R47, R48, R49, R50: symbol Device:R -> TMC51604Axis-rescue:R-Device
- TP3: symbol Connector:TestPoint -> TMC51604Axis-rescue:TestPoint-Connector
- U5, U6, U7: symbol 74xx:74LVC125 -> TMC51604Axis-rescue:74LVC125-74xx

Commit message: First layout V2
Parts:
- removed C44, C45: 100n, peters:C_0805_peter, symbol TMC51604Axis-rescue:C-Device
- removed D11, D12, D13, D14, D15, D16, D17, D18, D19: LED, peters:D_0805__HandSolder_peter, symbol TMC51604Axis-rescue:LED-Device
- removed D21, D22, D23, D24, D26, D29: BAT54S, Package_TO_SOT_SMD:SOT-23, symbol TMC51604Axis-rescue:BAT54S-Diode
- removed R41, R42, R43, R44, R45, R46, R47: 2k2, peters:R_0805_peter, symbol TMC51604Axis-rescue:R-Device
- removed R49: 100R, peters:R_0805_peter, symbol TMC51604Axis-rescue:R-Device
- removed R50: 20R, peters:R_0805_peter, symbol TMC51604Axis-rescue:R-Device
- removed unit 4 of U5
- removed U6, U7: 74LVC125, Package_SO:SO-14_5.3x10.2mm_P1.27mm, symbol TMC51604Axis-rescue:74LVC125-74xx
- added C2, C5: 100n, Capacitor_SMD:C_0603_1608Metric, symbol TMC51604Axis-rescue:C-Device
- added D11, D12, D13, D14, D16, D17, D18, D19: BAT54S, Package_TO_SOT_SMD:SOT-23, symbol TMC51604Axis-rescue:BAT54S-Diode
- added R1: 100R, peters:R_0805_peter, symbol TMC51604Axis-rescue:R-Device
- added R41: R, peters:C_0805_peter, symbol Device:R
- added U7: TXB0108PWR, digikey-footprints:TSSOP-20_W4.4mm, symbol dk_Logic-Translators-Level-Shifters:TXB0108PWR
- J3: value RJ45_Shielded -> RJ45_STEP_DIR
- J5: value RJ45_Shielded -> RJ45_SPI
- R31, R32: value 2k2 -> 100R
Connections:
- net +3V3: now also C5.2, U7.2 (VCCA)
- net CSN: now also U7.6 (A5)
- net CSN_raw: now also R39.1, D13.3, U7.15 (B5); no longer J5.2, R35.2
- net DIR_REFR: now also U7.5 (A4)
- net DRV_ENN: now also R32.1, D19.3
- net ENC_A_raw: now also D25.3, R40.2; no longer J4.2 (Pin_2), R38.2
- net ENC_B_raw: now also D27.3, R38.1; no longer J4.1 (Pin_1), R40.2
- net ENC_N_raw: now also D28.3; no longer J6.3 (Pin_3)
- net GND: now also J3.4, J3.6, J5.2, J5.4, J5.6, J5.8, C2.1, C5.1, D11.1, D12.1, D13.1, D14.1, D16.1, D17.1, D18.1, D19.1, R41.2, U7.11 (GND); no longer J3.1, J3.3, J3.5, J3.7, J5.1, J5.3, J5.5, J5.7
- net SCK: now also U7.9 (A8); no longer R31.1
- net SCK_raw: now also D20.3, R35.1, U7.12 (B8); no longer J5.8, R37.2
- net SDI: now also U7.7 (A6); no longer R32.1
- net SDI_raw: now also R37.1, D12.3, U7.14 (B6); no longer J5.4, R36.2
- net SDO: now also U7.8 (A7)
- net SDO_raw: now also R36.1, D11.3, U7.13 (B7); no longer J5.6, R34.2
- net STEP_REFL: now also U7.4 (A3)
- net at R32.2: now also J3.3
- net at R31.2: now also J3.5
- net DIAG0_SWn_OUT: now reaches R34.1
- net DIAG0_SWn_OUT: now also D18.3, U7.18 (B2)
- net DIAG1_SWp_OUT: now reaches R33.1
- net DIAG1_SWp_OUT: now also D17.3, U7.20 (B1); no longer D20.3
- net at R33.2: now also J3.2; no longer J3.4
- net at R39.2: now also J5.1; no longer J3.8
- net at R48.1: now also J6.3 (Pin_3); no longer D28.3
- net at R40.1: now also J4.2 (Pin_2); no longer D27.3
- net Signal_VCC renamed VBUS
- net VBUS: now also J3.8, C2.2, D11.2, D12.2, D13.2, D14.2, D16.2, D17.2, D18.2, D19.2, U7.19 (VCCB)
- new net: J4.1 (Pin_1), R38.2
- new net: J3.1, R34.2
- new net: J3.7, R1.2
- new net: J5.3, R37.2
- new net: J5.5, R36.2
- new net: J5.7, R35.2
- new net: R41.1, U7.10 (OE)
- new net DIAG0_SWn: U7.3 (A2)
- new net DIAG1_SWp: U7.1 (A1)
- new net DIR_raw: D14.3, R1.1, U7.16 (B4)
- new net Step_Raw: D16.3, R31.1, U7.17 (B3)
Other:
- note added: "SPI:\nCSN: ORG/WHT\nSDI: GRN/WHT\nSDO: BLU/WHT\nSCK: BRN/WHT"
- note added: "Step/Dir conn:\nDiag0: ORG/WHT\nDiag1: ORG\nDRVEna: GRN/WHT\nStep: BLU/WHT\nDir: BRN/WHT\nVBUS: BRN"
- moved on the sheet: C42, C46, C47, D20, J3, J5, R38, R40, R48, U5A, U5B, U5C
