File: TMC51604Axis/Inputs.sch (KiCad schematic (older format))
At the start: 39 parts, among them J3 RJ45_STEP_DIR, J4 EncCon1, J5 RJ45_SPI, J6 EncCon2, U5 74LVC125, U7 TXB0108PWR

Commit message: cleanup
Parts:
- added unit 4 of U5
Connections:
- net ENC_A: now also U5.5; no longer U5.6
- net ENC_A_raw: now also U5.6; no longer U5.5
- net GND: now also U5.11, U5.12, U5.13
Changed lines of the file:
@@
 F 1 "74LVC125" H 7530 3305 50  0000 L CNN
 F 2 "Package_SO:SO-14_5.3x10.2mm_P1.27mm" H 7300 3350 50  0001 C CNN
-F 3 "http://www.ti.com/lit/gpn/sn74LVC125" H 7300 3350 50  0001 C CNN
+F 3 "https://www.ti.com/lit/ds/symlink/sn74lvc125a.pdf?ts=1610054477145&ref_url=https%253A%252F%252Fwww.google.com%252F" H 7300 3350 50  0001 C CNN
 	5    7300 3350
 	1    0    0    -1
@@
 F 1 "74LVC125" H 8850 2876 50  0001 C CNN
 F 2 "Package_SO:SO-14_5.3x10.2mm_P1.27mm" H 8850 2650 50  0001 C CNN
-F 3 "http://www.ti.com/lit/gpn/sn74LVC125" H 8850 2650 50  0001 C CNN
+F 3 "https://www.ti.com/lit/ds/symlink/sn74lvc125a.pdf?ts=1610054477145&ref_url=https%253A%252F%252Fwww.google.com%252F" H 8850 2650 50  0001 C CNN
 	3    8850 2650
 	1    0    0    -1
@@
 $Comp
 L TMC51604Axis-rescue:74LVC125-74xx U?
+U 4 1 5FFC3458
+P 8850 3400
+AR Path="/5FFC3458" Ref="U?"  Part="3"
+AR Path="/5ED3D12E/5FFC3458" Ref="U5"  Part="4"
+F 0 "U5" H 8800 3400 50  0000 C CNN
+F 1 "74LVC125" H 8850 3626 50  0001 C CNN
+F 2 "Package_SO:SO-14_5.3x10.2mm_P1.27mm" H 8850 3400 50  0001 C CNN
+F 3 "https://www.ti.com/lit/ds/symlink/sn74lvc125a.pdf?ts=1610054477145&ref_url=https%253A%252F%252Fwww.google.com%252F" H 8850 3400 50  0001 C CNN
+	4    8850 3400
+	1    0    0    -1
+$EndComp
+$Comp
+L TMC51604Axis-rescue:GND-power #PWR?
+U 1 1 5FFC6319
+P 8850 3650
+AR Path="/5FFC6319" Ref="#PWR?"  Part="1"
+AR Path="/5ED3D12E/5FFC6319" Ref="#PWR?"  Part="1"
+F 0 "#PWR?" H 8850 3400 50  0001 C CNN
+F 1 "GND" H 8850 3500 50  0000 C CNN
+F 2 "" H 8850 3650 50  0001 C CNN
+F 3 "" H 8850 3650 50  0001 C CNN
+	1    8850 3650
+	1    0    0    -1
+$EndComp
+$Comp
+L TMC51604Axis-rescue:GND-power #PWR?
+U 1 1 5FFC67F5
+P 9150 3400
+AR Path="/5FFC67F5" Ref="#PWR?"  Part="1"
+AR Path="/5ED3D12E/5FFC67F5" Ref="#PWR?"  Part="1"
+F 0 "#PWR?" H 9150 3150 50  0001 C CNN
+F 1 "GND" H 9150 3250 50  0000 C CNN
+F 2 "" H 9150 3400 50  0001 C CNN
+F 3 "" H 9150 3400 50  0001 C CNN
+	1    9150 3400
+	1    0    0    -1
+$EndComp
+$Comp
+L TMC51604Axis-rescue:74LVC125-74xx U?
 U 1 1 5ED5E67B
 P 8850 2000
 AR Path="/5ED5E67B" Ref="U?"  Part="2"
 AR Path="/5ED3D12E/5ED5E67B" Ref="U5"  Part="1"
-F 0 "U5" H 8800 2000 50  0000 C CNN
+F 0 "U5" V 8800 2000 50  0000 C CNN
 F 1 "74LVC125" H 8850 2226 50  0001 C CNN
 F 2 "Package_SO:SO-14_5.3x10.2mm_P1.27mm" H 8850 2000 50  0001 C CNN
-F 3 "http://www.ti.com/lit/gpn/sn74LVC125" H 8850 2000 50  0001 C CNN
+F 3 "https://www.ti.com/lit/ds/symlink/sn74lvc125a.pdf?ts=1610054477145&ref_url=https%253A%252F%252Fwww.google.com%252F" H 8850 2000 50  0001 C CNN
 	1    8850 2000
 	1    0    0    -1
 $EndComp
-Wire Bus Line
-	3700 1900 3700 7100
-Wire Bus Line
-	2300 1100 2300 7100
 $Comp
 L TMC51604Axis-rescue:74LVC125-74xx U?
@@
 F 1 "74LVC125" H 8850 1576 50  0000 C CNN
 F 2 "Package_SO:SO-14_5.3x10.2mm_P1.27mm" H 8850 1350 50  0001 C CNN
-F 3 "http://www.ti.com/lit/gpn/sn74LVC125" H 8850 1350 50  0001 C CNN
+F 3 "https://www.ti.com/lit/ds/symlink/sn74lvc125a.pdf?ts=1610054477145&ref_url=https%253A%252F%252Fwww.google.com%252F" H 8850 1350 50  0001 C CNN
 	2    8850 1350
+	-1   0    0    -1
+$EndComp
+Wire Bus Line
+	2300 1100 2300 7100
+Wire Bus Line
+	3700 1900 3700 7100
+$Comp
+L TMC51604Axis-rescue:GND-power #PWR?
+U 1 1 6000AB21
+P 8550 3400
+AR Path="/6000AB21" Ref="#PWR?"  Part="1"
+AR Path="/5ED3D12E/6000AB21" Ref="#PWR?"  Part="1"
+F 0 "#PWR?" H 8550 3150 50  0001 C CNN
+F 1 "GND" H 8550 3250 50  0000 C CNN
+F 2 "" H 8550 3400 50  0001 C CNN
+F 3 "" H 8550 3400 50  0001 C CNN
+	1    8550 3400
 	1    0    0    -1
 $EndComp

Commit message: sync
Parts:
- R1, R31, R32, R33, R34, R35, R36, R37, R38, R39, R40, R48: footprint peters:R_0805_peter -> Resistor_SMD:R_0603_1608Metric
- R41: value R -> 62K
- U5: footprint Package_SO:SO-14_5.3x10.2mm_P1.27mm -> Package_SO:SO-14_3.9x8.65mm_P1.27mm
Connections:
- net +3V3: now also R41.1
- net GND: no longer R41.2, U5.11
- net at U7.10 (OE): now also R41.2; no longer R41.1
Other:
- moved on the sheet: R41
Changed lines of the file:
@@
 F 0 "U5" H 7530 3396 50  0000 L CNN
 F 1 "74LVC125" H 7530 3305 50  0000 L CNN
-F 2 "Package_SO:SO-14_5.3x10.2mm_P1.27mm" H 7300 3350 50  0001 C CNN
+F 2 "Package_SO:SO-14_3.9x8.65mm_P1.27mm" H 7300 3350 50  0001 C CNN
 F 3 "https://www.ti.com/lit/ds/symlink/sn74lvc125a.pdf?ts=1610054477145&ref_url=https%253A%252F%252Fwww.google.com%252F" H 7300 3350 50  0001 C CNN
 	5    7300 3350
@@
 F 0 "R38" V 7550 2200 50  0000 C CNN
 F 1 "100R" V 7450 2000 50  0000 C CNN
-F 2 "peters:R_0805_peter" V 7480 2000 50  0001 C CNN
+F 2 "Resistor_SMD:R_0603_1608Metric" V 7480 2000 50  0001 C CNN
 F 3 "~" H 7550 2000 50  0001 C CNN
 	1    7550 2000
@@
 F 0 "R48" V 7550 1900 50  0000 C CNN
 F 1 "100R" V 7550 2100 50  0000 C CNN
-F 2 "peters:R_0805_peter" V 7480 2100 50  0001 C CNN
+F 2 "Resistor_SMD:R_0603_1608Metric" V 7480 2100 50  0001 C CNN
 F 3 "~" H 7550 2100 50  0001 C CNN
 	1    7550 2100
@@
 F 0 "R40" V 7600 1700 50  0000 C CNN
 F 1 "100R" V 7434 1900 50  0000 C CNN
-F 2 "peters:R_0805_peter" V 7480 1900 50  0001 C CNN
+F 2 "Resistor_SMD:R_0603_1608Metric" V 7480 1900 50  0001 C CNN
 F 3 "~" H 7550 1900 50  0001 C CNN
 	1    7550 1900
@@
 F 0 "R31" V 1850 1200 50  0000 C CNN
 F 1 "100R" V 1950 1200 50  0000 C CNN
-F 2 "peters:R_0805_peter" V 1880 1200 50  0001 C CNN
+F 2 "Resistor_SMD:R_0603_1608Metric" V 1880 1200 50  0001 C CNN
 F 3 "~" H 1950 1200 50  0001 C CNN
 	1    1950 1200
@@
 F 0 "R1" V 1850 1000 50  0000 C CNN
 F 1 "100R" V 1950 1000 50  0000 C CNN
-F 2 "peters:R_0805_peter" V 1880 1000 50  0001 C CNN
+F 2 "Resistor_SMD:R_0603_1608Metric" V 1880 1000 50  0001 C CNN
 F 3 "~" H 1950 1000 50  0001 C CNN
 	1    1950 1000
@@
 F 0 "R32" V 1850 1400 50  0000 C CNN
 F 1 "100R" V 1950 1400 50  0000 C CNN
-F 2 "peters:R_0805_peter" V 1880 1400 50  0001 C CNN
+F 2 "Resistor_SMD:R_0603_1608Metric" V 1880 1400 50  0001 C CNN
 F 3 "~" H 1950 1400 50  0001 C CNN
 	1    1950 1400
@@
 F 0 "R33" V 2150 1500 50  0000 C CNN
 F 1 "100R" V 1950 1500 50  0000 C CNN
-F 2 "peters:R_0805_peter" V 1880 1500 50  0001 C CNN
+F 2 "Resistor_SMD:R_0603_1608Metric" V 1880 1500 50  0001 C CNN
 F 3 "~" H 1950 1500 50  0001 C CNN
 	1    1950 1500
@@
 F 0 "R34" V 2150 1600 50  0000 C CNN
 F 1 "100R" V 1950 1600 50  0000 C CNN
-F 2 "peters:R_0805_peter" V 1880 1600 50  0001 C CNN
+F 2 "Resistor_SMD:R_0603_1608Metric" V 1880 1600 50  0001 C CNN
 F 3 "~" H 1950 1600 50  0001 C CNN
 	1    1950 1600
@@
 F 0 "R35" V 2050 2950 50  0000 C CNN
 F 1 "100R" V 1950 2950 50  0000 C CNN
-F 2 "peters:R_0805_peter" V 1880 2950 50  0001 C CNN
+F 2 "Resistor_SMD:R_0603_1608Metric" V 1880 2950 50  0001 C CNN
 F 3 "~" H 1950 2950 50  0001 C CNN
 	1    1950 2950
@@
 F 0 "R36" V 2050 3150 50  0000 C CNN
 F 1 "100R" V 1950 3150 50  0000 C CNN
-F 2 "peters:R_0805_peter" V 1880 3150 50  0001 C CNN
+F 2 "Resistor_SMD:R_0603_1608Metric" V 1880 3150 50  0001 C CNN
 F 3 "~" H 1950 3150 50  0001 C CNN
 	1    1950 3150
@@
 F 0 "R37" V 2050 3350 50  0000 C CNN
 F 1 "100R" V 1950 3350 50  0000 C CNN
-F 2 "peters:R_0805_peter" V 1880 3350 50  0001 C CNN
+F 2 "Resistor_SMD:R_0603_1608Metric" V 1880 3350 50  0001 C CNN
 F 3 "~" H 1950 3350 50  0001 C CNN
 	1    1950 3350
@@
 F 0 "R39" V 2050 3550 50  0000 C CNN
 F 1 "100R" V 1950 3550 50  0000 C CNN
-F 2 "peters:R_0805_peter" V 1880 3550 50  0001 C CNN
+F 2 "Resistor_SMD:R_0603_1608Metric" V 1880 3550 50  0001 C CNN
 F 3 "~" H 1950 3550 50  0001 C CNN
 	1    1950 3550
@@
 L Device:R R41
 U 1 1 604F5AAB
-P 5100 3150
-F 0 "R41" H 5170 3196 50  0000 L CNN
-F 1 "R" H 5170 3105 50  0000 L CNN
-F 2 "peters:C_0805_peter" V 5030 3150 50  0001 C CNN
-F 3 "~" H 5100 3150 50  0001 C CNN
-	1    5100 3150
-	1    0    0    -1
-$EndComp
-$Comp
-L TMC51604Axis-rescue:GND-power #PWR?
-U 1 1 604F6153
-P 5100 3350
-AR Path="/604F6153" Ref="#PWR?"  Part="1"
-AR Path="/5ED3D12E/604F6153" Ref="#PWR0147"  Part="1"
-F 0 "#PWR0147" H 5100 3100 50  0001 C CNN
-F 1 "GND" H 5105 3177 50  0000 C CNN
-F 2 "" H 5100 3350 50  0001 C CNN
-F 3 "" H 5100 3350 50  0001 C CNN
-	1    5100 3350
-	1    0    0    -1
+P 5250 2800
+F 0 "R41" H 5320 2846 50  0000 L CNN
+F 1 "62K" H 5320 2755 50  0000 L CNN
+F 2 "peters:C_0805_peter" V 5180 2800 50  0001 C CNN
+F 3 "~" H 5250 2800 50  0001 C CNN
+	1    5250 2800
+	0    1    1    0
 $EndComp
 Wire Wire Line
-	5100 3350 5100 3300
-Wire Wire Line
 	5100 2800 5050 2800
 Wire Wire Line
-	5100 3000 5100 2800
-Wire Wire Line
 	5050 2000 5400 2000
 Wire Wire Line
@@
 F 0 "U5" H 8800 2650 50  0000 C CNN
 F 1 "74LVC125" H 8850 2876 50  0001 C CNN
-F 2 "Package_SO:SO-14_5.3x10.2mm_P1.27mm" H 8850 2650 50  0001 C CNN
+F 2 "Package_SO:SO-14_3.9x8.65mm_P1.27mm" H 8850 2650 50  0001 C CNN
 F 3 "https://www.ti.com/lit/ds/symlink/sn74lvc125a.pdf?ts=1610054477145&ref_url=https%253A%252F%252Fwww.google.com%252F" H 8850 2650 50  0001 C CNN
 	3    8850 2650
@@
 F 0 "U5" H 8800 3400 50  0000 C CNN
 F 1 "74LVC125" H 8850 3626 50  0001 C CNN
-F 2 "Package_SO:SO-14_5.3x10.2mm_P1.27mm" H 8850 3400 50  0001 C CNN
+F 2 "Package_SO:SO-14_3.9x8.65mm_P1.27mm" H 8850 3400 50  0001 C CNN
 F 3 "https://www.ti.com/lit/ds/symlink/sn74lvc125a.pdf?ts=1610054477145&ref_url=https%253A%252F%252Fwww.google.com%252F" H 8850 3400 50  0001 C CNN
 	4    8850 3400
@@
 $EndComp
 $Comp
-L TMC51604Axis-rescue:GND-power #PWR?
-U 1 1 5FFC67F5
-P 9150 3400
-AR Path="/5FFC67F5" Ref="#PWR?"  Part="1"
-AR Path="/5ED3D12E/5FFC67F5" Ref="#PWR0150"  Part="1"
-F 0 "#PWR0150" H 9150 3150 50  0001 C CNN
-F 1 "GND" H 9150 3250 50  0000 C CNN
-F 2 "" H 9150 3400 50  0001 C CNN
-F 3 "" H 9150 3400 50  0001 C CNN
-	1    9150 3400
-	1    0    0    -1
-$EndComp
-$Comp
 L TMC51604Axis-rescue:74LVC125-74xx U?
 U 1 1 5ED5E67B
@@
 F 0 "U5" V 8800 2000 50  0000 C CNN
 F 1 "74LVC125" H 8850 2226 50  0001 C CNN
-F 2 "Package_SO:SO-14_5.3x10.2mm_P1.27mm" H 8850 2000 50  0001 C CNN
+F 2 "Package_SO:SO-14_3.9x8.65mm_P1.27mm" H 8850 2000 50  0001 C CNN
 F 3 "https://www.ti.com/lit/ds/symlink/sn74lvc125a.pdf?ts=1610054477145&ref_url=https%253A%252F%252Fwww.google.com%252F" H 8850 2000 50  0001 C CNN
 	1    8850 2000
@@
 F 0 "U5" V 8800 1350 50  0000 C CNN
 F 1 "74LVC125" H 8850 1576 50  0000 C CNN
-F 2 "Package_SO:SO-14_5.3x10.2mm_P1.27mm" H 8850 1350 50  0001 C CNN
+F 2 "Package_SO:SO-14_3.9x8.65mm_P1.27mm" H 8850 1350 50  0001 C CNN
 F 3 "https://www.ti.com/lit/ds/symlink/sn74lvc125a.pdf?ts=1610054477145&ref_url=https%253A%252F%252Fwww.google.com%252F" H 8850 1350 50  0001 C CNN
 	2    8850 1350
 	-1   0    0    -1
 $EndComp
-Wire Bus Line
-	2300 1100 2300 7100
-Wire Bus Line
-	3700 1900 3700 7100
 $Comp
 L TMC51604Axis-rescue:GND-power #PWR?
@@
 	1    0    0    -1
 $EndComp
+Wire Bus Line
+	2300 1100 2300 7100
+Wire Bus Line
+	3700 1900 3700 7100
+$Comp
+L TMC51604Axis-rescue:+3.3V-Peters #PWR?
+U 1 1 6025209F
+P 5400 2800
+AR Path="/6025209F" Ref="#PWR?"  Part="1"
+AR Path="/5ED3D12E/6025209F" Ref="#PWR0147"  Part="1"
+F 0 "#PWR0147" H 5400 2650 50  0001 C CNN
+F 1 "+3.3V" H 5415 2973 50  0000 C CNN
+F 2 "" H 5400 2800 50  0001 C CNN
+F 3 "" H 5400 2800 50  0001 C CNN
+	1    5400 2800
+	0    1    1    0
+$EndComp
 $EndSCHEMATC
