File: TMC51604Axis/MotorDrv1.sch (KiCad schematic (older format))
At the start: 62 parts

Commit message: Sync
Parts:
- removed C?: 220uF/100V, symbol Device:CP
- removed D? (x4): 1A/60V, symbol Device:D_Schottky_Small
- removed D? (x8): DNP, symbol Device:D_Schottky_Small
- removed Q? (x2): DMHT6016LFJ, symbol Peters:DMHT6016LFJ
- added C21: 220uF/100V, Capacitor_THT:C_Radial_D16.0mm_H25.0mm_P7.50mm, symbol Device:CP
- added D1, D11, D12, D2, D5, D6, D7, D8: BAT54, digikey-footprints:SOT-23-3, symbol dk_Diodes-Rectifiers-Single:BAT54
- added D10, D3, D4, D9: ZHCS1006TA, Package_TO_SOT_SMD:SOT-23_Handsoldering, symbol Peters:ZHCS1006TA
- added Q2, Q3: DMHT6016LFJ, Libs:V-DFN5045-12, symbol Peters:DMHT6016LFJ
- C1: renamed from C?; footprint (none) -> Capacitor_SMD:C_1210_3225Metric_Pad1.42x2.65mm_HandSolder
- C10, C2, C3: renamed from C?; footprint (none) -> Capacitor_SMD:C_0805_2012Metric_Pad1.15x1.40mm_HandSolder
- C11, C12, C13, C14, C19, C22, C23, C24, C4, C5, C8, C9: renamed from C?; footprint (none) -> Capacitor_SMD:C_0603_1608Metric_Pad1.05x0.95mm_HandSolder
- C15, C16, C17, C18, C20, C6: renamed from C?; footprint (none) -> Capacitor_SMD:C_1206_3216Metric_Pad1.42x1.75mm_HandSolder
- C7: renamed from C?; footprint (none) -> Capacitor_THT:C_Radial_D16.0mm_H25.0mm_P7.50mm
- R1: renamed from R?; footprint (none) -> Resistor_SMD:R_1210_3225Metric_Pad1.42x2.65mm_HandSolder
- R10, R19: renamed from R?; footprint (none) -> Resistor_SMD:R_2512_6332Metric_Pad1.52x3.35mm_HandSolder
- R11, R12, R13, R14, R15, R16, R17, R18, R2, R20, R21, R22, R3, R4, R5, R6, R7, R8, R9: renamed from R?; footprint (none) -> Resistor_SMD:R_0805_2012Metric_Pad1.15x1.40mm_HandSolder
- U1: renamed from U?; footprint eTQFP48_9x9 -> Package_QFP:TQFP-48-1EP_7x7mm_P0.5mm_EP5x5mm_ThermalVias
- gave numbers to parts that had none: 1
Connections:
- wire segments 191 -> 193
Other:
- moved on the sheet: R10, R11, R18, R19, R20, R9

Commit message: sync
Parts:
- removed D1, D11, D12, D2, D5, D6, D7, D8: BAT54, digikey-footprints:SOT-23-3, symbol dk_Diodes-Rectifiers-Single:BAT54
- C10, C2: footprint Capacitor_SMD:C_0805_2012Metric_Pad1.15x1.40mm_HandSolder -> Capacitor_SMD:C_0603_1608Metric
- C11, C12, C13, C14, C19, C22, C23, C24, C4, C5, C8, C9: footprint Capacitor_SMD:C_0603_1608Metric_Pad1.05x0.95mm_HandSolder -> Capacitor_SMD:C_0603_1608Metric
- C15, C16, C17, C18, C20, C6: footprint Capacitor_SMD:C_1206_3216Metric_Pad1.42x1.75mm_HandSolder -> Capacitor_SMD:C_1206_3216Metric
- D10, D3, D4, D9: footprint Package_TO_SOT_SMD:SOT-23_Handsoldering -> Package_TO_SOT_SMD:SOT-23
- R1: footprint Resistor_SMD:R_1210_3225Metric_Pad1.42x2.65mm_HandSolder -> Resistor_SMD:R_1210_3225Metric
- R10, R19: footprint Resistor_SMD:R_2512_6332Metric_Pad1.52x3.35mm_HandSolder -> Resistor_SMD:R_2512_6332Metric
- R11, R12, R13, R14, R15, R16, R17, R18, R2, R20, R21, R22, R3, R4, R5, R6, R7, R8, R9: footprint Resistor_SMD:R_0805_2012Metric_Pad1.15x1.40mm_HandSolder -> Resistor_SMD:R_0603_1608Metric_Pad1.05x0.95mm_HandSolder
- U1: symbol 2019-09-25_19-26-57:TMC5160-TA -> TMC51604Axis-rescue:TMC5160-TA-2019-09-25_19-26-57
Connections:
- wire segments 193 -> 177

Commit message: Layout done! Still untested
Parts:
- removed U1: TMC5160-TA, Package_QFP:TQFP-48-1EP_7x7mm_P0.5mm_EP5x5mm_ThermalVias, symbol TMC51604Axis-rescue:TMC5160-TA-2019-09-25_19-26-57
- added C15: 100n/100v, Capacitor_SMD:C_1210_3225Metric_Pad1.42x2.65mm_HandSolder, symbol Device:C_Small
- added C34: 100n, Capacitor_SMD:C_0603_1608Metric, symbol Device:C_Small
- added C37: 15pF, peters:D_0805_peter, symbol Device:C
- added JP1: SPI_MODE, Jumper:SolderJumper-3_P2.0mm_Open_TrianglePad1.0x1.5mm, symbol Device:Jumper_NC_Dual
- added JP2: SD_MODE, Jumper:SolderJumper-3_P2.0mm_Open_TrianglePad1.0x1.5mm, symbol Device:Jumper_NC_Dual
- added R18: 100k, peters:R_0805_peter, symbol Device:R
- added R19: NC, peters:R_0805_peter, symbol Device:R
- added U3: TMC5160A-TA, peters:LQFP-48-1EP_7x7mm_P0.5mm_EP3.6x3.6mm_peter, symbol Peters:TMC5160A-TA
- added U4: ASDMB-12.0MHz, Oscillator:Oscillator_SMD_Abracon_ASDMB-4Pin_2.5x2.0mm, symbol Oscillator:ASDMB-xxxMHz
- C16: renamed from C1; value 4,7uF -> 4,7uF/100v
- C18: renamed from C3; footprint Capacitor_SMD:C_0805_2012Metric_Pad1.15x1.40mm_HandSolder -> peters:C_0805_peter
- C19: renamed from C4; value 220n -> 220n/100v
- C21: renamed from C7; footprint Capacitor_THT:C_Radial_D16.0mm_H25.0mm_P7.50mm -> Capacitor_SMD:CP_Elec_10x14.3
- C23: renamed from C8; value 10uF -> 2.2uF
- C28: renamed from C15; footprint Capacitor_SMD:C_1206_3216Metric -> Capacitor_SMD:C_0603_1608Metric
- C29: renamed from C16; footprint Capacitor_SMD:C_1206_3216Metric -> Capacitor_SMD:C_0603_1608Metric
- C30: renamed from C17; footprint Capacitor_SMD:C_1206_3216Metric -> Capacitor_SMD:C_0603_1608Metric
- C31: renamed from C18; footprint Capacitor_SMD:C_1206_3216Metric -> Capacitor_SMD:C_0603_1608Metric
- C39: renamed from C21; footprint Capacitor_THT:C_Radial_D16.0mm_H25.0mm_P7.50mm -> Capacitor_SMD:CP_Elec_10x14.3
- R10: renamed from R2; footprint Resistor_SMD:R_0603_1608Metric_Pad1.05x0.95mm_HandSolder -> Resistor_SMD:R_0603_1608Metric
- R11: renamed from R3; footprint Resistor_SMD:R_0603_1608Metric_Pad1.05x0.95mm_HandSolder -> Resistor_SMD:R_0603_1608Metric
- R12: renamed from R8; footprint Resistor_SMD:R_0603_1608Metric_Pad1.05x0.95mm_HandSolder -> Resistor_SMD:R_0603_1608Metric
- R13: renamed from R4; footprint Resistor_SMD:R_0603_1608Metric_Pad1.05x0.95mm_HandSolder -> Resistor_SMD:R_0603_1608Metric
- R14: renamed from R5; footprint Resistor_SMD:R_0603_1608Metric_Pad1.05x0.95mm_HandSolder -> Resistor_SMD:R_0603_1608Metric
- R15: renamed from R9; footprint Resistor_SMD:R_0603_1608Metric_Pad1.05x0.95mm_HandSolder -> Resistor_SMD:R_0603_1608Metric
- R16: renamed from R10; footprint Resistor_SMD:R_2512_6332Metric -> Resistor_SMD:R_1206_3216Metric
- R17: renamed from R11; footprint Resistor_SMD:R_0603_1608Metric_Pad1.05x0.95mm_HandSolder -> Resistor_SMD:R_0603_1608Metric
- R20: renamed from R16; footprint Resistor_SMD:R_0603_1608Metric_Pad1.05x0.95mm_HandSolder -> Resistor_SMD:R_0603_1608Metric
- R21: renamed from R17; footprint Resistor_SMD:R_0603_1608Metric_Pad1.05x0.95mm_HandSolder -> Resistor_SMD:R_0603_1608Metric
- R22: renamed from R12; footprint Resistor_SMD:R_0603_1608Metric_Pad1.05x0.95mm_HandSolder -> Resistor_SMD:R_0603_1608Metric
- R23: renamed from R13; footprint Resistor_SMD:R_0603_1608Metric_Pad1.05x0.95mm_HandSolder -> Resistor_SMD:R_0603_1608Metric
- R24: renamed from R14; footprint Resistor_SMD:R_0603_1608Metric_Pad1.05x0.95mm_HandSolder -> Resistor_SMD:R_0603_1608Metric
- R25: renamed from R15; footprint Resistor_SMD:R_0603_1608Metric_Pad1.05x0.95mm_HandSolder -> Resistor_SMD:R_0603_1608Metric
- R26: renamed from R18; footprint Resistor_SMD:R_0603_1608Metric_Pad1.05x0.95mm_HandSolder -> Resistor_SMD:R_0603_1608Metric
- R27: renamed from R19; footprint Resistor_SMD:R_2512_6332Metric -> Resistor_SMD:R_1206_3216Metric
- R28: renamed from R20; footprint Resistor_SMD:R_0603_1608Metric_Pad1.05x0.95mm_HandSolder -> Resistor_SMD:R_0603_1608Metric
- R29: renamed from R21; footprint Resistor_SMD:R_0603_1608Metric_Pad1.05x0.95mm_HandSolder -> Resistor_SMD:R_0603_1608Metric
- R30: renamed from R22; footprint Resistor_SMD:R_0603_1608Metric_Pad1.05x0.95mm_HandSolder -> Resistor_SMD:R_0603_1608Metric
- R7: renamed from R1; footprint Resistor_SMD:R_1210_3225Metric -> peters:R_0805_peter
- R8: renamed from R6; footprint Resistor_SMD:R_0603_1608Metric_Pad1.05x0.95mm_HandSolder -> Resistor_SMD:R_0603_1608Metric
- R9: renamed from R7; footprint Resistor_SMD:R_0603_1608Metric_Pad1.05x0.95mm_HandSolder -> Resistor_SMD:R_0603_1608Metric
- renumbered C2 to C17, C6 to C20, C5 to C22, C9 to C24, C10 to C25, C11 to C26, C12 to C27, C13 to C32, C14 to C33, C19 to C35, C22 to C36, C20 to C38, C23 to C40, C24 to C41, D3 to D7, D4 to D8
Connections:
- net labels added: DIAG0_SWn, DIAG1_SWp, REFL_STEP, REFR_DIR, VCC_IO, VMotor, VSA
- net labels removed: +12V, +VMotor
- wire segments 177 -> 195
Other:
- note added: "A minimum capacity of 100µF per ampere of coil current near to the power\nbridge is recommended for best performance."
- note added: "opt. ext. clock 12-16MHz\npage 118 of TMC5160 DATASHEET\n (Rev. 1.10 / 2019-FEB-05) 118\n"
- note removed: "Filter capacitors placed near bridge"
- note removed: "opt. ext. clock 12-16MHz\npage 118 of TMC5160 DATASHEET (Rev. 1.10 / 2019-FEB-05) 118\n"

Commit message: Redone input section
Parts:
- added R51, R52: 0R1, Resistor_SMD:R_1206_3216Metric, symbol Device:R
Connections:
- wire segments 195 -> 203
Other:
- moved on the sheet: R15, R16, R17, R18, R19, R26, R27, R28, U3

Commit message: Bug fixes during first assembly
Parts:
- C15, C16, C17, C19, C22, C23, C24, C25, C26, C27, C32, C33, C34, C35, C36, C40, C41: symbol Device:C_Small -> TMC51604Axis-rescue:C_Small-Device
- C18: footprint peters:C_0805_peter -> Capacitor_SMD:C_0603_1608Metric; symbol Device:C_Small -> TMC51604Axis-rescue:C_Small-Device
- C20, C28, C29, C30, C31, C37, C38: symbol Device:C -> TMC51604Axis-rescue:C-Device
- C21, C39: symbol Device:CP -> TMC51604Axis-rescue:CP-Device
- D10, D7, D8, D9: symbol Peters:ZHCS1006TA -> TMC51604Axis-rescue:ZHCS1006TA-Peters
- JP1, JP2: symbol Device:Jumper_NC_Dual -> TMC51604Axis-rescue:Jumper_NC_Dual-Device
- Q2, Q3: symbol Peters:DMHT6016LFJ -> TMC51604Axis-rescue:DMHT6016LFJ-Peters
- Q4: symbol Transistor_FET:BSS138 -> TMC51604Axis-rescue:BSS138-Transistor_FET
- R10, R11, R12, R13, R14, R20, R21, R22, R23, R24, R25, R29, R30, R7, R8, R9: symbol Device:R_Small -> TMC51604Axis-rescue:R_Small-Device
- R15, R16, R17, R18, R19, R26, R27, R28, R51, R52: symbol Device:R -> TMC51604Axis-rescue:R-Device
- U3: symbol Peters:TMC5160A-TA -> TMC51604Axis-rescue:TMC5160A-TA-Peters
- U4: symbol Oscillator:ASDMB-xxxMHz -> TMC51604Axis-rescue:ASDMB-xxxMHz-Oscillator

Commit message: First layout V2
Parts:
- removed C21, C39: 220uF/100V, Capacitor_SMD:CP_Elec_10x14.3, symbol TMC51604Axis-rescue:CP-Device
- removed R51, R52: 0R1, Resistor_SMD:R_1206_3216Metric, symbol TMC51604Axis-rescue:R-Device
- added C50, C51: 470n/100V, Capacitor_SMD:C_1206_3216Metric, symbol TMC51604Axis-rescue:C-Device
- added C52, C53, C54, C55: 330uF/100V, Capacitor_THT:CP_Radial_D12.5mm_P5.00mm, symbol TMC51604Axis-rescue:CP-Device
- added Q1: BSS138, Package_TO_SOT_SMD:SOT-23, symbol TMC51604Axis-rescue:BSS138-Transistor_FET
- added R42, R43, R44: 100K, Resistor_SMD:R_0603_1608Metric, symbol TMC51604Axis-rescue:R_Small-Device
- added R45, R46: 10K, Resistor_SMD:R_0603_1608Metric, symbol TMC51604Axis-rescue:R_Small-Device
- added R53, R54: 47K, Resistor_SMD:R_0603_1608Metric, symbol TMC51604Axis-rescue:R_Small-Device
- C15, C16: footprint Capacitor_SMD:C_1210_3225Metric_Pad1.42x2.65mm_HandSolder -> Capacitor_SMD:C_1210_3225Metric_Pad1.33x2.70mm_HandSolder
- C17: Digikery partno (none) -> 445-2275-1-ND
- C20, C38: value 470n/100V -> 470n/100V x2
- C23: value 2.2uF -> 2.2uFto10uF
- C25: value 2.2u -> 2.2uFto10uF
- JP1, JP2: footprint Jumper:SolderJumper-3_P2.0mm_Open_TrianglePad1.0x1.5mm -> Jumper:SolderJumper-3_P1.3mm_Bridged12_RoundedPad1.0x1.5mm
- Q2, Q3: value DMHT6016LFJ -> DMHT6016LFJ-Peters; footprint Libs:V-DFN5045-12 -> Libs:V-DFN5045-12 (Type B)
- R16, R27: value 0R1 -> 0R05; footprint Resistor_SMD:R_1206_3216Metric -> Resistor_SMD:R_2512_6332Metric_Pad1.40x3.35mm_HandSolder
- R19: footprint peters:R_0805_peter -> Resistor_SMD:R_0603_1608Metric
Connections:
- net labels added: SDI, SDO, SD_MODE, SPI_MODE, SRA+, SRA-, SRB+, SRB-
- net labels removed: MISO, MOSI
- wire segments 203 -> 226
Other:
- note added: "Make sure that VSA does not drop out during\nmotor operation. The motor driver should be disabled in case VSA becomes switched off before VS."
- note added: "Mount pullups when used as linit switches"
- note added: "Use C37 footprint as pulldown if osc. not in use"
- note added: "Use low inductivity SMD type, e.g. 1210 or 2512 resistor for RS!\nPage 74 TMC5160 DATASHEET (Rev. 1.14 / 2020-MAY-19)"
- note added: "VCC:\nWhen using an external\nsupply, make sure, that VCC comes up before or in parallel to\n5VOUT or VCC_IO, whichever comes up later!"
- note removed: "Use low inductivity SMD type, e.g. 1210 or 2512 resistor for RS!\nPage 73 TMC5160 DATASHEET (Rev. 1.10 / 2019-FEB-05)"
- moved on the sheet: C20, C23, C27, C32, C34, C37, C38, C40, JP1, Q4, R13, R14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

Commit message: cleanup
Parts:
- C15, C16: footprint Capacitor_SMD:C_1210_3225Metric_Pad1.33x2.70mm_HandSolder -> Capacitor_SMD:C_1206_3216Metric
Changed lines of the file:
@@
 F 0 "C15" V 7250 1900 50  0000 L CNN
 F 1 "100n/100v" V 7300 2150 50  0000 L CNN
-F 2 "Capacitor_SMD:C_1210_3225Metric_Pad1.33x2.70mm_HandSolder" H 7300 1850 50  0001 C CNN
+F 2 "Capacitor_SMD:C_1206_3216Metric" H 7300 1850 50  0001 C CNN
 F 3 "~" H 7300 1850 50  0001 C CNN
 	1    7300 1850
@@
 F 0 "C16" V 7500 1900 50  0000 L CNN
 F 1 "4,7uF/100v" V 7550 2150 50  0000 L CNN
-F 2 "Capacitor_SMD:C_1210_3225Metric_Pad1.33x2.70mm_HandSolder" H 7550 1850 50  0001 C CNN
+F 2 "Capacitor_SMD:C_1206_3216Metric" H 7550 1850 50  0001 C CNN
 F 3 "~" H 7550 1850 50  0001 C CNN
 	1    7550 1850

Commit message: correced silk top
Parts:
- C19: footprint Capacitor_SMD:C_0603_1608Metric -> Capacitor_SMD:C_0805_2012Metric
Changed lines of the file:
@@
 F 0 "C19" V 7300 2200 50  0000 L CNN
 F 1 "220n/100v" V 7250 1800 50  0000 L CNN
-F 2 "Capacitor_SMD:C_0603_1608Metric" H 7150 2350 50  0001 C CNN
+F 2 "Capacitor_SMD:C_0805_2012Metric" H 7150 2350 50  0001 C CNN
 F 3 "~" H 7150 2350 50  0001 C CNN
 	1    7150 2350
