File: TMC51604Axis/MotorDrv1.sch (KiCad schematic (older format))
At the start: 74 parts, among them Q1 BSS138, Q2 DMHT6016LFJ-Peters, Q3 DMHT6016LFJ-Peters, Q4 BSS138, U3 TMC5160A-TA, U4 ASDMB-12.0MHz

Commit message: sync
Parts:
- removed D10, D7, D8, D9: ZHCS1006TA, Package_TO_SOT_SMD:SOT-23, symbol TMC51604Axis-rescue:ZHCS1006TA-Peters
- added D10, D7, D8, D9: PMEG6010CEGWX, Diode_SMD:D_SOD-123, symbol Device:D_Schottky_Small_ALT
Connections:
- net GND: now also D10.2 (A), D7.2 (A), D8.2 (A), D9.2 (A)
- net at R9.1, U3.48 (BMB1): now also D9.1 (K)
- net at R12.1, U3.45 (BMB2): now also D7.1 (K)
- net at R20.1, U3.40 (BMA1): now also D10.1 (K)
- net at R21.1, U3.37 (BMA2): now also D8.1 (K)
Other:
- moved on the sheet: C22, C24, C26, C35, C36, R12, R20, R21, R9
